Commit message: Started to update URDF with STL models

File: src/robot_decapsuleur/urdf/robot.urdf (robot description, URDF)
Before this commit: robot my_robot, 4 links, 3 joints
Links:
- removed link arriere_bras
- removed link avant_bras
- removed link rotatif
- added link arm1; visual mesh filename=package://robot_decapsuleur/stl/arm.STL scale=0.01 0.01 0.01
- added link base2; visual mesh filename=package://robot_decapsuleur/stl/base_plate-2.STL scale=0.01 0.01 0.01
- added link dyna1; visual mesh filename=package://robot_decapsuleur/stl/DYNAMIXEL_AX-12A.STL scale=0.01 0.01 0.01
- added link dyna2; visual mesh filename=package://robot_decapsuleur/stl/DYNAMIXEL_AX-12A.STL scale=0.01 0.01 0.01
- added link rot; visual mesh filename=package://robot_decapsuleur/stl/Rotating_plate.STL scale=0.01 0.01 0.01
- link base: geometry visual mesh filename=package://robot_decapsuleur/stl/base_plate-1.STL scale=0.01 0.01 0.01
Joints:
- added joint joint3: type fixed, parent rot, child dyna2, origin xyz=0 0 0 rpy=0 0 0
- added joint joint4: type continuous, parent dyna2, child arm1, origin xyz=1 1 -1 rpy=0 0 0
- joint joint0: axis 0 0 1 -> (none); child rotatif -> base2; origin xyz=0 0 2 rpy=0 0 0 -> xyz=0 0 0.63 rpy=0 0 0; type continuous -> fixed
- joint joint1: axis 1 0 0 -> (none); child arriere_bras -> dyna1; origin xyz=0 0 3 rpy=0 0 0 -> xyz=0 0 -0.15 rpy=0 0 0; parent rotatif -> base2; type continuous -> fixed
- joint joint2: axis 1 0 0 -> 0 0 1; child avant_bras -> rot; origin xyz=0 0 3 rpy=0 0 0 -> xyz=0 0 0.185 rpy=0 0 0; parent arriere_bras -> dyna1

Commit message: Finalized first prototype of urdf

File: src/robot_decapsuleur/urdf/robot.urdf (robot description, URDF)
Before this commit: robot my_robot, 6 links, 5 joints
Links:
- added link arm2; visual mesh filename=package://robot_decapsuleur/stl/arm.STL scale=0.01 0.01 0.01
- added link dyna3; visual mesh filename=package://robot_decapsuleur/stl/DYNAMIXEL_AX-12A.STL scale=0.01 0.01 0.01
Joints:
- added joint joint5: type fixed, parent arm1, child dyna3, origin xyz=0 0 0 rpy=0 0 0
- added joint joint6: type continuous, parent dyna3, child arm2, origin xyz=0 0 2.09 rpy=0 0 0
- joint joint4: origin xyz=1 1 -1 rpy=0 0 0 -> xyz=0.55 0.175 0.205 rpy=0 0 0
