Commit message: Renamed robot_decapsuleur to robot_decapsuleur_description

File: src/robot_decapsuleur_description/urdf/robot.urdf (robot description, URDF)
Before this commit: robot my_robot, 8 links, 7 joints
Links:
- link arm1: geometry visual mesh filename=package://robot_decapsuleur_description/stl/arm.STL scale=0.01 0.01 0.01
- link arm2: geometry visual mesh filename=package://robot_decapsuleur_description/stl/arm.STL scale=0.01 0.01 0.01
- link base: geometry visual mesh filename=package://robot_decapsuleur_description/stl/base_plate-1.STL scale=0.01 0.01 0.01
- link base2: geometry visual mesh filename=package://robot_decapsuleur_description/stl/base_plate-2.STL scale=0.01 0.01 0.01
- link dyna1: geometry visual mesh filename=package://robot_decapsuleur_description/stl/DYNAMIXEL_AX-12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 scale=0.01 0.01 0.01
- link dyna2: geometry visual mesh filename=package://robot_decapsuleur_description/stl/DYNAMIXEL_AX-12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 scale=0.01 0.01 0.01
- link dyna3: geometry visual mesh filename=package://robot_decapsuleur_description/stl/DYNAMIXEL_AX-12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 scale=0.01 0.01 0.01
- link rot: geometry visual mesh filename=package://robot_decapsuleur_description/stl/Rotating_plate.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 scale=0.01 0.01 0.01
