Commit message: Renamed robot to robot_decapsuleur + added few functionnalities (sleep and cap frame)

File: src/robot_decapsuleur_description/urdf/robot.urdf.xacro (robot description, xacro)
@@ -1,3 +1,3 @@
-<robot name="my_robot">
+<robot name="robot_decapsuleur">
 	<link name="base">
 		<visual>
@@ -67,5 +67,5 @@
 		<visual>
 			<geometry>
-				<box size="0.9 1.8 0.1"/>
+				<box size="1.0 2.95 0.05"/>
 			</geometry>
 			<origin rpy="${-pi/2} 0 0" xyz="0 0 0"/>
@@ -77,5 +77,5 @@
 				<mesh filename="package://robot_decapsuleur_description/stl/rplidar_a2.stl" scale="0.01 0.01 0.01"/>
 			</geometry>
-			<origin rpy="${pi/2} ${pi/2} 0" xyz="-0.25 0 0"/>
+			<origin rpy="0 0 ${-pi/2}" xyz="-0.25 0 0"/>
 		</visual>
 	</link>
@@ -86,4 +86,20 @@
 			</geometry>
 			<origin rpy="0 ${pi/2} ${pi}" xyz="0 0 0"/>
+		</visual>
+	</link>
+	<link name="bottle_opener_support">
+		<visual>
+			<geometry>
+				<mesh filename="package://robot_decapsuleur_description/stl/bottle_opener_support.stl" scale="0.01 0.01 0.01"/>
+			</geometry>
+			<origin rpy="0 ${pi/2} 0" xyz="0 0 0"/>
+		</visual>
+	</link>
+	<link name="bottle_opener">
+		<visual>
+			<geometry>
+				<mesh filename="package://robot_decapsuleur_description/stl/bottle_opener.stl" scale="0.01 0.01 0.01"/>
+			</geometry>
+			<origin rpy="${pi/2} 0 0" xyz="0 0 0"/>
 		</visual>
 	</link>
@@ -127,10 +143,10 @@
 		<parent link="arm2"/>
 		<child link="lidar_support"/>
-		<origin rpy="0 0 0" xyz="0 -0.25 0.1"/>
+		<origin rpy="0 0 0" xyz="0 -0.32 -0.1"/>
 	</joint>
 	<joint name="joint_lidar" type="fixed">
 		<parent link="lidar_support"/>
 		<child link="lidar"/>
-		<origin rpy="0 0 0" xyz="0 -0.05 -0.3"/>
+		<origin rpy="${pi/2} 0 0" xyz="0 -0.05 -0.93"/>
 	</joint>
 	<joint name="joint_arm5" type="fixed">
@@ -139,3 +155,13 @@
 		<origin rpy="0 0 0" xyz="0 0 2.09"/>
 	</joint>
+	<joint name="joint_arm6" type="continuous">
+		<parent link="dyna4"/>
+		<child link="bottle_opener_support"/>
+		<origin rpy="${-pi/2} 0 0" xyz="0 0 0"/>
+	</joint>
+	<joint name="joint_arm7" type="fixed">
+		<parent link="bottle_opener_support"/>
+		<child link="bottle_opener"/>
+		<origin rpy="0 0 0" xyz="0 -0.25 -0.2"/>
+	</joint>
 </robot>

Commit message: Added moveit and fixed URDF

File: src/robot_decapsuleur_description/urdf/robot.urdf.xacro (robot description, xacro)
@@ -1,3 +1,4 @@
 <robot name="robot_decapsuleur">
+	<link name="base_link" />
 	<link name="base">
 		<visual>
@@ -37,5 +38,5 @@
 				<mesh filename="package://robot_decapsuleur_description/stl/DYNAMIXEL_AX-12A.STL" scale="0.01 0.01 0.01"/>
 			</geometry>
-			<origin rpy="${pi/2} 0 ${-pi/2}" xyz="0.008 0.175 0.205"/>
+			<origin rpy="${pi/2} 0 ${pi/2}" xyz="0.008 0.175 0.205"/>
 		</visual>
 	</link>
@@ -45,5 +46,5 @@
 				<mesh filename="package://robot_decapsuleur_description/stl/arm.STL" scale="0.01 0.01 0.01"/>
 			</geometry>
-			<origin rpy="${pi/2} ${-pi/2} 0" xyz="0.565 1.435 -0.755"/>
+			<origin rpy="${pi/2} ${-pi/2} ${pi}" xyz="-0.565 -1.435 -0.755"/>
 		</visual>
 	</link>
@@ -53,5 +54,5 @@
 				<mesh filename="package://robot_decapsuleur_description/stl/DYNAMIXEL_AX-12A.STL" scale="0.01 0.01 0.01"/>
 			</geometry>
-			<origin rpy="0 ${pi/2} ${pi}" xyz="0 0 0"/>
+			<origin rpy="${pi/2} ${pi/2} ${-pi/2}" xyz="0 0 0"/>
 		</visual>
 	</link>
@@ -61,5 +62,5 @@
 				<mesh filename="package://robot_decapsuleur_description/stl/arm.STL" scale="0.01 0.01 0.01"/>
 			</geometry>
-			<origin rpy="${pi/2} ${-pi/2} 0" xyz="0.565 1.435 -0.755"/>
+			<origin rpy="${pi/2} ${-pi/2} ${pi}" xyz="-0.565 -1.435 -0.755"/>
 		</visual>
 	</link>
@@ -104,4 +105,8 @@
 		</visual>
 	</link>
+	<joint name="joint_base_link" type="fixed">
+		<parent link="base_link"/>
+		<child link="base"/>
+	</joint>
 	<joint name="joint_base1" type="fixed">
 		<parent link="base"/>
@@ -117,5 +122,5 @@
 		<parent link="dyna1"/>
 		<child link="rot"/>
-		<origin rpy="0 0 0" xyz="0 0 0.185"/>
+		<origin rpy="0 0 ${pi/2 + pi/4}" xyz="0 0 0.185"/>
 		<axis xyz="0 0 1" />
 	</joint>
@@ -123,25 +128,25 @@
 		<parent link="rot"/>
 		<child link="dyna2"/>
-		<origin rpy="0 0 0" xyz="0 0 0"/>
+		<origin rpy="0 0 ${pi}" xyz="0 0.28 0"/>
 	</joint>
 	<joint name="joint_arm2" type="continuous">
 		<parent link="dyna2"/>
 		<child link="arm1"/>
-		<origin rpy="0 0 0" xyz="0 0.175 0.205"/>
+		<origin rpy="${pi/2} 0 0" xyz="0 0.175 0.205"/>
 	</joint>
 	<joint name="joint_arm3" type="fixed">
 		<parent link="arm1"/>
 		<child link="dyna3"/>
-		<origin rpy="0 0 0" xyz="0 0 2.09"/>
+		<origin rpy="0 0 ${pi}" xyz="0 0 2.09"/>
 	</joint>
 	<joint name="joint_arm4" type="continuous">
 		<parent link="dyna3"/>
 		<child link="arm2"/>
-		<origin rpy="0 0 0" xyz="0 0 0"/>
+		<origin rpy="${-pi/2} ${pi} 0" xyz="0 0 0"/>
 	</joint>
 	<joint name="joint_lidar_support" type="fixed">
 		<parent link="arm2"/>
 		<child link="lidar_support"/>
-		<origin rpy="0 0 0" xyz="0 -0.32 -0.1"/>
+		<origin rpy="0 0 ${pi}" xyz="0 0.32 -0.1"/>
 	</joint>
 	<joint name="joint_lidar" type="fixed">

Commit message: Improved overall performances and fixed bugs

File: src/robot_decapsuleur_description/urdf/robot.urdf.xacro (robot description, xacro)
@@ -4,5 +4,5 @@
 		<visual>
 			<geometry>
-				<mesh filename="package://robot_decapsuleur_description/stl/base_plate-1.STL" scale="0.01 0.01 0.01"/>
+				<mesh filename="package://robot_decapsuleur_description/stl/base_plate-1.dae" scale="0.01 0.01 0.01"/>
 			</geometry>
 		  <origin rpy="0 0 0" xyz="-0.6 -0.6 0"/>
@@ -12,5 +12,5 @@
 		<visual>
 			<geometry>
-				<mesh filename="package://robot_decapsuleur_description/stl/base_plate-2.STL" scale="0.01 0.01 0.01"/>
+				<mesh filename="package://robot_decapsuleur_description/stl/base_plate-2.dae" scale="0.01 0.01 0.01"/>
 			</geometry>
 			<origin rpy="0 0 0" xyz="-0.45 -0.45 0"/>
@@ -20,5 +20,5 @@
 		<visual>
 			<geometry>
-				<mesh filename="package://robot_decapsuleur_description/stl/DYNAMIXEL_AX-12A.STL" scale="0.01 0.01 0.01"/>
+				<mesh filename="package://robot_decapsuleur_description/stl/DYNAMIXEL_AX-12A.dae" scale="0.01 0.01 0.01"/>
 			</geometry>
 			<origin rpy="0 0 ${-pi/2}" xyz="0 0 0"/>
@@ -28,5 +28,5 @@
 		<visual>
 			<geometry>
-				<mesh filename="package://robot_decapsuleur_description/stl/Rotating_plate.STL" scale="0.01 0.01 0.01"/>
+				<mesh filename="package://robot_decapsuleur_description/stl/Rotating_plate.dae" scale="0.01 0.01 0.01"/>
 			</geometry>
 			<origin rpy="0 0 0.1" xyz="-0.4 -0.5 0"/>
@@ -36,5 +36,5 @@
 		<visual>
 			<geometry>
-				<mesh filename="package://robot_decapsuleur_description/stl/DYNAMIXEL_AX-12A.STL" scale="0.01 0.01 0.01"/>
+				<mesh filename="package://robot_decapsuleur_description/stl/DYNAMIXEL_AX-12A.dae" scale="0.01 0.01 0.01"/>
 			</geometry>
 			<origin rpy="${pi/2} 0 ${pi/2}" xyz="0.008 0.175 0.205"/>
@@ -44,5 +44,5 @@
 		<visual>
 			<geometry>
-				<mesh filename="package://robot_decapsuleur_description/stl/arm.STL" scale="0.01 0.01 0.01"/>
+				<mesh filename="package://robot_decapsuleur_description/stl/arm.dae" scale="0.01 0.01 0.01"/>
 			</geometry>
 			<origin rpy="${pi/2} ${-pi/2} ${pi}" xyz="-0.565 -1.435 -0.755"/>
@@ -52,5 +52,5 @@
 		<visual>
 			<geometry>
-				<mesh filename="package://robot_decapsuleur_description/stl/DYNAMIXEL_AX-12A.STL" scale="0.01 0.01 0.01"/>
+				<mesh filename="package://robot_decapsuleur_description/stl/DYNAMIXEL_AX-12A.dae" scale="0.01 0.01 0.01"/>
 			</geometry>
 			<origin rpy="${pi/2} ${pi/2} ${-pi/2}" xyz="0 0 0"/>
@@ -60,5 +60,5 @@
 		<visual>
 			<geometry>
-				<mesh filename="package://robot_decapsuleur_description/stl/arm.STL" scale="0.01 0.01 0.01"/>
+				<mesh filename="package://robot_decapsuleur_description/stl/arm.dae" scale="0.01 0.01 0.01"/>
 			</geometry>
 			<origin rpy="${pi/2} ${-pi/2} ${pi}" xyz="-0.565 -1.435 -0.755"/>
@@ -76,5 +76,5 @@
 		<visual>
 			<geometry>
-				<mesh filename="package://robot_decapsuleur_description/stl/rplidar_a2.stl" scale="0.01 0.01 0.01"/>
+				<mesh filename="package://robot_decapsuleur_description/stl/rplidar_a2.dae" scale="0.01 0.01 0.01"/>
 			</geometry>
 			<origin rpy="0 0 ${-pi/2}" xyz="-0.25 0 0"/>
@@ -84,5 +84,5 @@
 		<visual>
 			<geometry>
-				<mesh filename="package://robot_decapsuleur_description/stl/DYNAMIXEL_AX-12A.STL" scale="0.01 0.01 0.01"/>
+				<mesh filename="package://robot_decapsuleur_description/stl/DYNAMIXEL_AX-12A.dae" scale="0.01 0.01 0.01"/>
 			</geometry>
 			<origin rpy="0 ${pi/2} ${pi}" xyz="0 0 0"/>
@@ -92,5 +92,5 @@
 		<visual>
 			<geometry>
-				<mesh filename="package://robot_decapsuleur_description/stl/bottle_opener_support.stl" scale="0.01 0.01 0.01"/>
+				<mesh filename="package://robot_decapsuleur_description/stl/bottle_opener_support.dae" scale="0.01 0.01 0.01"/>
 			</geometry>
 			<origin rpy="0 ${pi/2} 0" xyz="0 0 0"/>
@@ -100,5 +100,5 @@
 		<visual>
 			<geometry>
-				<mesh filename="package://robot_decapsuleur_description/stl/bottle_opener.stl" scale="0.01 0.01 0.01"/>
+				<mesh filename="package://robot_decapsuleur_description/stl/bottle_opener.dae" scale="0.01 0.01 0.01"/>
 			</geometry>
 			<origin rpy="${pi/2} 0 0" xyz="0 0 0"/>
@@ -163,5 +163,5 @@
 		<parent link="dyna4"/>
 		<child link="bottle_opener_support"/>
-		<origin rpy="${-pi/2} 0 0" xyz="0 0 0"/>
+		<origin rpy="${pi/2} ${pi} 0" xyz="0 0 0"/>
 	</joint>
 	<joint name="joint_arm7" type="fixed">
